File: CAN.kicad_sch (KiCad schematic)
At the start: 2 parts, among them J401 RJ45_Shielded, J402 RJ45_Shielded

Commit message: almost finished
Parts:
- J401, J402: footprint MFP19RJ45:RJ45_YH59_01 -> KicadZeniteSolarLibrary18:RJ45_YH59_01
Changed lines of the file:
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@@
       (effects (font (size 1.27 1.27)) (justify right))
     )
-    (property "Footprint" "MFP19RJ45:RJ45_YH59_01" (id 2) (at 120.65 74.295 90)
+    (property "Footprint" "KicadZeniteSolarLibrary18:RJ45_YH59_01" (id 2) (at 120.65 74.295 90)
       (effects (font (size 1.27 1.27)) hide)
     )
@@
       (effects (font (size 1.27 1.27)) (justify right))
     )
-    (property "Footprint" "MFP19RJ45:RJ45_YH59_01" (id 2) (at 157.48 74.295 90)
+    (property "Footprint" "KicadZeniteSolarLibrary18:RJ45_YH59_01" (id 2) (at 157.48 74.295 90)
       (effects (font (size 1.27 1.27)) hide)
     )
