File: supply1.kicad_sch (KiCad schematic)
At the start: 26 parts, among them Q1 Si2308CDS, U1 LMR16030

Commit message: almost finished
Parts:
- added D201: MBR340, Diode_SMD:D_SMA_Handsoldering, symbol Device:D_Schottky
Connections:
- net +18V: now also D201.1 (K)
- net CAN_18V_DIODE renamed LED
- net LED: now also D201.2 (A)
Changed lines of the file:
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@@
   (junction (at 110.49 85.09) (diameter 0) (color 0 0 0 0)
   )
+  (junction (at 219.71 62.23) (diameter 0) (color 0 0 0 0)
+  )
   (junction (at 128.27 55.88) (diameter 0) (color 0 0 0 0)
+  )
+  (junction (at 212.09 62.23) (diameter 0) (color 0 0 0 0)
   )
   (junction (at 184.15 85.09) (diameter 0) (color 0 0 0 0)
@@
     (stroke (width 0) (type default) (color 0 0 0 0))
   )
+  (wire (pts (xy 212.09 62.23) (xy 212.09 64.77))
+    (stroke (width 0) (type default) (color 0 0 0 0))
+  )
   (wire (pts (xy 156.21 85.09) (xy 160.02 85.09))
     (stroke (width 0) (type default) (color 0 0 0 0))
@@
   )
   (wire (pts (xy 166.37 62.23) (xy 168.91 62.23))
+    (stroke (width 0) (type default) (color 0 0 0 0))
+  )
+  (wire (pts (xy 219.71 62.23) (xy 219.71 64.77))
     (stroke (width 0) (type default) (color 0 0 0 0))
   )
@@
   (hierarchical_label "IN" (shape input) (at 67.31 69.85 180)
     (effects (font (size 1.27 1.27)) (justify right))
+  )
+  (hierarchical_label "LED" (shape input) (at 199.39 52.07 0)
+    (effects (font (size 1.27 1.27)) (justify left))
   )
   (hierarchical_label "GND" (shape input) (at 212.09 85.09 0)
@@
     (pin "1")
   )
+  (symbol (lib_id "Device:D_Schottky") (at 215.9 64.77 180) (unit 1)
+    (in_bom yes) (on_board yes)
+    (property "Reference" "D201" (id 0) (at 215.9 69.85 0))
+    (property "Value" "MBR340" (id 1) (at 215.9 67.31 0))
+    (property "Footprint" "Diode_SMD:D_SMA_Handsoldering" (id 2) (at 215.9 64.77 0)
+      (effects (font (size 1.27 1.27)) hide)
+    )
+    (property "Datasheet" "~" (id 3) (at 215.9 64.77 0)
+      (effects (font (size 1.27 1.27)) hide)
+    )
+    (pin "1")
+    (pin "2")
+  )
   (symbol (lib_id "fonte_18V-rescue:C_Small-Device") (at 200.66 73.66 0) (unit 1)
